Commit message: Update arm.urdf.xacro
Change made to the camera_link

File: arm_description/urdf/arm.urdf.xacro (robot description, xacro)
@@ -361,6 +361,6 @@
       <visual>
         <geometry>
-          <box size="0.01 0.01 0.01"/>
-          <!--mesh filename="package://arm_description/meshes/YASHICA_ELECTRO_35.stl" scale="0.0003 0.0003 0.0003"/-->
+          <!--box size="0.01 0.01 0.01"/-->
+          <mesh filename="package://arm_description/meshes/YASHICA_ELECTRO_35.stl" scale="0.0003 0.0003 0.0003"/>
         </geometry>
         <origin rpy="0 0 1.571" xyz="0.015 0 -0.02"/>
