Commit message: Update arm.urdf

File: arm_description/urdf/arm.urdf (robot description, URDF)
Before this commit: robot arm, 17 links, 16 joints
Links:
- link base_link: geometry collision box size=0.09 0.09 0.0975; visual mesh filename=package://arm_description/meshes/base_link.stl scale=0.001 0.001 0.001
- link base_turn: geometry collision box size=0.062 0.079 0.007; visual mesh filename=package://arm_description/meshes/base_turn.stl scale=0.001 0.001 0.001
- link base_turn_rot: geometry collision cylinder length=0.022 radius=0.0285; visual mesh filename=package://arm_description/meshes/base_turn_table_rot.stl scale=0.001 0.001 0.001
- link crawer_base: geometry collision box size=0.11 0.058 0.005; visual mesh filename=package://arm_description/meshes/the_crawer_base.stl scale=0.001 0.001 0.001
- link crawer_left: geometry collision cylinder length=0.056 radius=0.027; visual mesh filename=package://arm_description/meshes/the_crawer.stl scale=0.001 0.001 0.001
- link crawer_right: geometry collision cylinder length=0.056 radius=0.027; visual mesh filename=package://arm_description/meshes/the_crawer.stl scale=0.001 0.001 0.001
- link dyn2: geometry collision box size=0.051 0.032 0.042; visual mesh filename=package://arm_description/meshes/dyn.stl scale=0.01 0.01 0.01
- link dyn3: geometry collision box size=0.051 0.032 0.042; visual mesh filename=package://arm_description/meshes/dyn.stl scale=0.01 0.01 0.01
- link dyn4: geometry collision box size=0.051 0.032 0.042; visual mesh filename=package://arm_description/meshes/dyn.stl scale=0.01 0.01 0.01
- link dyn5: geometry collision box size=0.051 0.032 0.042; visual mesh filename=package://arm_description/meshes/dyn.stl scale=0.01 0.01 0.01
- link f4: geometry collision box size=0.05 0.061 0.03; visual mesh filename=package://arm_description/meshes/f4_n_f3.stl scale=0.001 0.001 0.001
- link f5: geometry collision box size=0.05 0.061 0.03; visual mesh filename=package://arm_description/meshes/f4_n_f3.stl scale=0.001 0.001 0.001
- link wrist: geometry collision box size=0.049 0.055 0.017; visual mesh filename=package://arm_description/meshes/wrist.stl scale=0.001 0.001 0.001
